Commit message: dolly v1 urdf update

File: catkin_ws/dolly/urdf/dolly.urdf (robot description, URDF)
Before this commit: robot ASM_Ver_1.SLDASM, 3 links, 2 joints
Links:
- removed link base
- added link base_link, mass 2.75822986493914; collision mesh filename=package://dolly/meshes/base_link.STL; visual mesh filename=package://dolly/meshes/base_link.STL
- link left_wheel: mass 0.2139 -> 0.21389788050971; geometry collision mesh filename=package://dolly/meshes/left_wheel.STL; visual mesh filename=package://dolly/meshes/left_wheel.STL
- link right_wheel: mass 0.2139 -> 0.21389788050971; geometry collision mesh filename=package://dolly/meshes/right_wheel.STL; visual mesh filename=package://dolly/meshes/right_wheel.STL
Joints:
- joint left_wheel_to_base: parent base -> base_link
- joint right_wheel_to_base: parent base -> base_link
