Commit message: Now dolly description lies in dolly_description, not just in dolly

File: catkin_ws/src/dolly_description/urdf/dolly.urdf (robot description, URDF)
Before this commit: robot dolly, 5 links, 4 joints
Links:
- link back_caster: geometry collision mesh filename=package://dolly_description/meshes/back_caster.STL; visual mesh filename=package://dolly_description/meshes/back_caster.STL
- link base_link: geometry collision mesh filename=package://dolly_description/meshes/base_link.STL; visual mesh filename=package://dolly_description/meshes/base_link.STL
- link front_caster: geometry collision mesh filename=package://dolly_description/meshes/front_caster.STL; visual mesh filename=package://dolly_description/meshes/front_caster.STL
- link left_wheel: geometry collision mesh filename=package://dolly_description/meshes/left_wheel.STL; visual mesh filename=package://dolly_description/meshes/left_wheel.STL
- link right_wheel: geometry collision mesh filename=package://dolly_description/meshes/right_wheel.STL; visual mesh filename=package://dolly_description/meshes/right_wheel.STL

Commit message: Added non inertial root link in urdf robot description

File: catkin_ws/src/dolly_description/urdf/dolly.urdf (robot description, URDF)
Before this commit: robot dolly, 5 links, 4 joints
Links:
- added link base_footprint; visual cylinder length=0.001 radius=0.1
Joints:
- added joint base_link_to_footprint: type continuous, parent base_footprint, child base_link, origin xyz=0 0 0.016 rpy=0 0 0, axis 0 -1 0

Commit message: dolly_description package is ready: simple rviz driving

File: catkin_ws/src/dolly_description/urdf/dolly.urdf (robot description, URDF)
Before this commit: robot dolly, 6 links, 5 joints
Joints:
- removed joint base_link_to_footprint
- added joint base_footprint_to_base_link: type fixed, parent base_footprint, child base_link, origin xyz=0 0 0.016 rpy=0 0 0, axis 0 -1 0
