Commit message: Night before competition

File: catkin_ws/src/dolly_description/urdf/dolly_description.urdf (robot description, URDF)
Before this commit: robot dolly_description, 6 links, 5 joints
Links:
- added link sensors; visual box size=0.03 0.03 0.03
Joints:
- added joint sensors_to_base: type fixed, parent base_link, child sensors, origin xyz=0 0 0 rpy=0 0 0, axis 0 0 0
