Commit message: modified aruco description files

File: catkin_ws/src/aruco_description/urdf/general_aruco.urdf.xacro (robot description, xacro)
@@ -4,5 +4,5 @@
     <xacro:arg name="aruco_id" default="0"/>
     <xacro:arg name="aruco_name" default="DICT_4X4_100_id0"/>
-    <xacro:arg name="aruco_l" default="0.2"/>
+    <xacro:arg name="aruco_l" default="0.1"/>
     <xacro:arg name="white_border" default="0"/>
     <xacro:arg name="meshes_directory" default="$(find aruco_description)/meshes"/>

File: catkin_ws/src/aruco_description/urdf/general_aruco.xacro (robot description, xacro)
@@ -24,5 +24,5 @@
         <origin xyz="0 0 0" rpy="0 0 0"/>
         <geometry>
-          <box size="${aruco_l + 2*white_border * aruco_l} ${aruco_l + 2*white_border * aruco_l} ${0.01 * aruco_l/0.09}"/>
+          <box size="${aruco_l} ${aruco_l} ${aruco_l}"/>
         </geometry>
       </collision>
@@ -38,5 +38,5 @@
           <!-- <box size="0.09 0.09 0.01"/> -->
           <!-- <mesh filename="package://aruco_description/meshes/${aruco_dictionary}/${aruco_dictionary}_id${aruco_id}.dae" scale="${aruco_l/0.09} ${aruco_l/0.09} ${aruco_l/0.09}"/> -->
-          <mesh filename="${meshes_directory}/${aruco_dictionary}/${aruco_dictionary}_id${aruco_id}.dae" scale="${aruco_l/0.09} ${aruco_l/0.09} ${aruco_l*0/0.09}"/>
+          <mesh filename="${meshes_directory}/${aruco_dictionary}/${aruco_dictionary}_id${aruco_id}.dae" scale="${aruco_l/0.09} ${aruco_l/0.09} ${aruco_l*0/0.01}"/>
         </geometry>
       </visual>
